File: Z680 Subwoofer/Z680 Standalone Subwoofer/Z680 Standalone Subwoofer.kicad_pcb (KiCad board)
At the start: 2 copper layers, 72 x 32 mm, 14 parts, among them J1 Conn_Coaxial, J2 DB15_Female_HighDensity, U1 MC78M05_TO252

Commit message: Reupload Kicad Files
Reupload kicad files in response to issue #1
Other:
- net class Default removed

Commit message: Revision 1
Fix low end gain on volume
Parts:
- added R4: 10k, Resistor_SMD:R_0603_1608Metric, F.Cu at (60.0, 28.2)
- J2: footprint Connector_Dsub:DSUB-15-HD_Female_Vertical_P2.29x1.98mm_MountingHoles -> Connector_Dsub:DSUB-15-HD_Socket_Vertical_P2.29x1.98mm_MountingHoles
- R3: footprint Capacitor_SMD:C_0805_2012Metric -> Resistor_SMD:R_0805_2012Metric
- moved U1 0.90 mm to (22.8, 32.0)
Routing:
- net /SGND: track 14.7 -> 19.0 mm, vias 161 -> 162
- net /DGND: track 19.3 -> 21.8 mm
- net /Sub_Input: track 38.8 -> 40.5 mm
Other:
- board text added: "Z680 Standalone Subwoofer R${REVISION}-BDM-${ISSUE_DATE} CC BY-SA 4.0 License"
- board text removed: "Z680 Standalone Subwoofer BDM 2021-10-27 CC BY-SA 4.0 License"
